File: hacks/dra818v_breakout_board/dra818v_breakout_board.kicad_pcb (KiCad board)
At the start: 2 copper layers, 48.3 x 30.8 mm, 4 parts

Commit message: finished v01 and ordered pcb
Parts:
- C1: value (none) -> 100nF X7R
- J1: value (none) -> SMA female
- P1: value (none) -> CONN_01X10
- U1: value (none) -> DRA818V
Connections:
- U1 pad 11: Net-(U1-Pad11) -> (no net)
- U1 pad 13: Net-(U1-Pad13) -> (no net)
- U1 pad 14: Net-(U1-Pad14) -> (no net)
- U1 pad 15: Net-(U1-Pad15) -> (no net)
- U1 pad 2: Net-(U1-Pad2) -> (no net)
- U1 pad 4: Net-(U1-Pad4) -> (no net)
Routing:
- net GND: track 0.00 -> 67.7 mm
- net Net-(P1-Pad10): track 0.00 -> 43.3 mm, vias 0 -> 1
- net Net-(P1-Pad9): track 0.00 -> 36.4 mm, vias 0 -> 1
- net VCC: track 0.00 -> 33.4 mm
- net Net-(P1-Pad8): track 0.00 -> 28.1 mm, vias 0 -> 1
- net Net-(P1-Pad3): track 0.00 -> 22.7 mm
- net Net-(P1-Pad5): track 0.00 -> 18.2 mm
- net Net-(P1-Pad4): track 0.00 -> 17.5 mm
- net Net-(J1-Pad1): track 0.00 -> 11.8 mm
- net Net-(P1-Pad2): track 0.00 -> 9.38 mm
- net Net-(P1-Pad1): track 0.00 -> 5.53 mm
- added copper zone on B.Cu, net GND
- added copper zone on F.Cu, net GND
Other:
- board size 48.3 x 30.8 mm -> 48.3 x 30.7 mm
- rule pad_to_mask_clearance: 0.2 -> 0.076
- board text added: "DRA818 breakout board v0.1 By @mik4el4ndersson 2016"
